Commit message: update

File: gogogo/src/unitree_ros/robots/g1_description/g1_23dof.urdf (robot description, URDF)
Before this commit: robot g1_23dof, 30 links, 29 joints
Links:
- removed link imu_link
- added link d435_link
- added link imu_in_pelvis
- added link imu_in_torso
- added link mid360_link
Joints:
- removed joint imu_joint
- added joint d435_joint: type fixed, parent torso_link, child d435_link, origin xyz=0.0576235 0.01753 0.41987 rpy=0 0.8307767239493009 0
- added joint imu_in_pelvis_joint: type fixed, parent pelvis, child imu_in_pelvis, origin xyz=0.04525 0 -0.08339 rpy=0 0 0
- added joint imu_in_torso_joint: type fixed, parent torso_link, child imu_in_torso, origin xyz=-0.03959 -0.00224 0.13792 rpy=0 0 0
- added joint mid360_joint: type fixed, parent torso_link, child mid360_link, origin xyz=0.0002835 0.00003 0.40618 rpy=0 0.04014257279586953 0

File: gogogo/src/unitree_ros/robots/g1_description/g1_29dof.urdf (robot description, URDF)
Before this commit: robot g1_29dof, 37 links, 36 joints
Links:
- removed link imu_link
- added link d435_link
- added link imu_in_pelvis
- added link imu_in_torso
- added link mid360_link
Joints:
- removed joint imu_joint
- added joint d435_joint: type fixed, parent torso_link, child d435_link, origin xyz=0.0576235 0.01753 0.41987 rpy=0 0.8307767239493009 0
- added joint imu_in_pelvis_joint: type fixed, parent pelvis, child imu_in_pelvis, origin xyz=0.04525 0 -0.08339 rpy=0 0 0
- added joint imu_in_torso_joint: type fixed, parent torso_link, child imu_in_torso, origin xyz=-0.03959 -0.00224 0.13792 rpy=0 0 0
- added joint mid360_joint: type fixed, parent torso_link, child mid360_link, origin xyz=0.0002835 0.00003 0.40618 rpy=0 0.04014257279586953 0

File: gogogo/src/unitree_ros/robots/g1_description/g1_29dof_with_hand.urdf (robot description, URDF)
Before this commit: robot g1_29dof_with_hand, 51 links, 50 joints
Links:
- removed link imu_link
- added link d435_link
- added link imu_in_pelvis
- added link imu_in_torso
- added link mid360_link
- link left_hand_index_0_link: mass 0.05619628 -> 0.05885070
- link left_hand_index_1_link: mass 0.02487314 -> 0.02030626
- link left_hand_middle_0_link: mass 0.05619628 -> 0.05885070
- link left_hand_middle_1_link: mass 0.02487314 -> 0.02030626
- link left_hand_thumb_0_link: mass 0.08033018 -> 0.08623657
- link left_hand_thumb_1_link: mass 0.05619628 -> 0.05885070
- link left_hand_thumb_2_link: mass 0.02487314 -> 0.02030626
- link right_hand_index_0_link: mass 0.05619628 -> 0.05885070
- link right_hand_index_1_link: mass 0.02487314 -> 0.02030626
- link right_hand_middle_0_link: mass 0.05619628 -> 0.05885070
- link right_hand_middle_1_link: mass 0.02487314 -> 0.02030626
- link right_hand_thumb_0_link: mass 0.08033018 -> 0.08623657
- link right_hand_thumb_1_link: mass 0.05619628 -> 0.05885070
- link right_hand_thumb_2_link: mass 0.02487314 -> 0.02030626
Joints:
- removed joint imu_joint
- added joint d435_joint: type fixed, parent torso_link, child d435_link, origin xyz=0.0576235 0.01753 0.41987 rpy=0 0.8307767239493009 0
- added joint imu_in_pelvis_joint: type fixed, parent pelvis, child imu_in_pelvis, origin xyz=0.04525 0 -0.08339 rpy=0 0 0
- added joint imu_in_torso_joint: type fixed, parent torso_link, child imu_in_torso, origin xyz=-0.03959 -0.00224 0.13792 rpy=0 0 0
- added joint mid360_joint: type fixed, parent torso_link, child mid360_link, origin xyz=0.0002835 0.00003 0.40618 rpy=0 0.04014257279586953 0
- joint left_hand_index_0_joint: limit lower=-1.83259571 upper=0.19198621 effort=0.7 velocity=24 -> lower=-1.57079632 upper=0 effort=1.4 velocity=12; origin xyz=0.1 -0.0017 0.0285 rpy=0 0 0 -> xyz=0.0777 0.0016 0.0285 rpy=0 0 0
- joint left_hand_index_1_joint: limit lower=-2.09439510 upper=0 effort=0.7 velocity=24 -> lower=-1.74532925 upper=0 effort=1.4 velocity=12; origin xyz=0.0528 -0.0055 0 rpy=0 0 0 -> xyz=0.0458 0 0 rpy=0 0 0
- joint left_hand_middle_0_joint: limit lower=-1.83259571 upper=0.19198621 effort=0.7 velocity=24 -> lower=-1.57079632 upper=0 effort=1.4 velocity=12; origin xyz=0.1 -0.0017 -0.0285 rpy=0 0 0 -> xyz=0.0777 0.0016 -0.0285 rpy=0 0 0
- joint left_hand_middle_1_joint: limit lower=-2.09439510 upper=0 effort=0.7 velocity=24 -> lower=-1.74532925 upper=0 effort=1.4 velocity=12; origin xyz=0.0528 -0.0055 0 rpy=0 0 0 -> xyz=0.0458 0 0 rpy=0 0 0
- joint left_hand_thumb_0_joint: origin xyz=0.028 0 0 rpy=0 0 0 -> xyz=0.0255 0 0 rpy=0 0 0
- joint left_hand_thumb_1_joint: limit lower=-0.72431163 upper=1.04719755 effort=0.7 velocity=24 -> lower=-0.72431163 upper=1.04719755 effort=1.4 velocity=12; origin xyz=0 -0.0246 0 rpy=0 0 0 -> xyz=-0.0025 -0.0193 0 rpy=0 0 0
- joint left_hand_thumb_2_joint: limit lower=0 upper=2.09439510 effort=0.7 velocity=24 -> lower=0 upper=1.74532925 effort=1.4 velocity=12; origin xyz=0.0055 -0.0528 0 rpy=0 0 0 -> xyz=0 -0.0458 0 rpy=0 0 0
- joint right_hand_index_0_joint: limit lower=-0.19198621 upper=1.83259571 effort=0.7 velocity=24 -> lower=0 upper=1.57079632 effort=1.4 velocity=12; origin xyz=0.1 0.0017 0.0285 rpy=0 0 0 -> xyz=0.0777 -0.0016 0.0285 rpy=0 0 0
- joint right_hand_index_1_joint: limit lower=0 upper=2.09439510 effort=0.7 velocity=24 -> lower=0 upper=1.74532925 effort=1.4 velocity=12; origin xyz=0.0528 0.0055 0 rpy=0 0 0 -> xyz=0.0458 0 0 rpy=0 0 0
- joint right_hand_middle_0_joint: limit lower=-0.19198621 upper=1.83259571 effort=0.7 velocity=24 -> lower=0 upper=1.57079632 effort=1.4 velocity=12; origin xyz=0.1 0.0017 -0.0285 rpy=0 0 0 -> xyz=0.0777 -0.0016 -0.0285 rpy=0 0 0
- joint right_hand_middle_1_joint: limit lower=0 upper=2.09439510 effort=0.7 velocity=24 -> lower=0 upper=1.74532925 effort=1.4 velocity=12; origin xyz=0.0528 0.0055 0 rpy=0 0 0 -> xyz=0.0458 0 0 rpy=0 0 0
- joint right_hand_thumb_0_joint: origin xyz=0.028 0 0 rpy=0 0 0 -> xyz=0.0255 0 0 rpy=0 0 0
- joint right_hand_thumb_1_joint: limit lower=-1.04719755 upper=0.72431163 effort=0.7 velocity=24 -> lower=-1.04719755 upper=0.72431163 effort=1.4 velocity=12; origin xyz=0 0.0246 0 rpy=0 0 0 -> xyz=-0.0025 0.0193 0 rpy=0 0 0
- joint right_hand_thumb_2_joint: limit lower=-2.09439510 upper=0 effort=0.7 velocity=24 -> lower=-1.74532925 upper=0 effort=1.4 velocity=12; origin xyz=0.0055 0.0528 0 rpy=0 0 0 -> xyz=0 0.0458 0 rpy=0 0 0

File: gogogo/src/unitree_ros/robots/g1_description/g1_dual_arm.urdf (robot description, URDF)
Before this commit: robot g1_dual_arm, 23 links, 22 joints
Links:
- removed link imu_link
- added link d435_link
- added link imu_in_pelvis
- added link imu_in_torso
- added link mid360_link
Joints:
- removed joint imu_joint
- added joint d435_joint: type fixed, parent torso_link, child d435_link, origin xyz=0.0576235 0.01753 0.41987 rpy=0 0.8307767239493009 0
- added joint imu_in_pelvis_joint: type fixed, parent pelvis, child imu_in_pelvis, origin xyz=0.04525 0 -0.08339 rpy=0 0 0
- added joint imu_in_torso_joint: type fixed, parent torso_link, child imu_in_torso, origin xyz=-0.03959 -0.00224 0.13792 rpy=0 0 0
- added joint mid360_joint: type fixed, parent torso_link, child mid360_link, origin xyz=0.0002835 0.00003 0.40618 rpy=0 0.04014257279586953 0

File: gogogo/src/unitree_ros/robots/go1_description/xacro/depthCamera.xacro (robot description, xacro)
@@ -45,6 +45,6 @@
                     </image>
                     <clip>
-                        <near>0.05</near>
-                        <far>8</far>
+                        <near>0.1</near>
+                        <far>5</far>
                     </clip>
                 </camera>

File: gogogo/src/unitree_ros/robots/go1_description/xacro/gazebo.xacro (robot description, xacro)
@@ -9,5 +9,5 @@
     </gazebo>
     <!-- Show the trajectory of trunk center. -->
-    <!-- <gazebo>
+    <gazebo>
         <plugin name="3dplot" filename="libLinkPlot3DPlugin.so">
             <frequency>10</frequency>
@@ -18,5 +18,5 @@
             </plot>
         </plugin>
-    </gazebo> -->
+    </gazebo>
     <!-- Show the trajectory of foot. You can add another trajectory about another foot. -->
     <!-- <gazebo>

File: gogogo/src/unitree_ros/robots/go1_description/xacro/robot.xacro (robot description, xacro)
@@ -88,5 +88,5 @@
     <xacro:leg name="RL" mirror="1"  mirror_dae="True"   front_hind="-1" front_hind_dae="False" />
     <xacro:depthCamera camID="1" name="face">
-        <origin rpy="0 0 0" xyz="0.27 0.0 0.03"/>
+        <origin rpy="${PI} 0 0" xyz="0.2785 0.0125 0.0167"/>
     </xacro:depthCamera>
     <xacro:depthCamera camID="2" name="chin">
